File: KiCAD/ADC1.sch (KiCad schematic (older format))
At the start: 27 parts, among them J1 Conn_02x08_Odd_Even, J2 Conn_02x08_Odd_Even, J3 Conn_02x08_Odd_Even, J4 Conn_02x08_Odd_Even, J53 Conn_02x10_Odd_Even, U1 AD7779

Commit message: Add files via upload
Changed lines of the file:
@@
 AR Path="/5CE92453/5CDD1CC4" Ref="C43"  Part="1"
 AR Path="/5CE92455/5CDD1CC4" Ref="C64"  Part="1"
-F 0 "C1" H 3292 2996 50  0000 L CNN
+F 0 "C22" H 3292 2996 50  0000 L CNN
 F 1 "100n" H 3292 2905 50  0000 L CNN
 F 2 "Capacitor_SMD:C_0402_1005Metric" H 3200 2950 50  0001 C CNN
@@
 AR Path="/5CE92453/5CDD1CCB" Ref="C45"  Part="1"
 AR Path="/5CE92455/5CDD1CCB" Ref="C66"  Part="1"
-F 0 "C3" H 3292 3496 50  0000 L CNN
+F 0 "C24" H 3292 3496 50  0000 L CNN
 F 1 "100n" H 3292 3405 50  0000 L CNN
 F 2 "Capacitor_SMD:C_0402_1005Metric" H 3200 3450 50  0001 C CNN
@@
 AR Path="/5CE92453/5CDD1CD2" Ref="C44"  Part="1"
 AR Path="/5CE92455/5CDD1CD2" Ref="C65"  Part="1"
-F 0 "C2" H 3642 2996 50  0000 L CNN
+F 0 "C23" H 3642 2996 50  0000 L CNN
 F 1 "1u" H 3642 2905 50  0000 L CNN
 F 2 "Capacitor_SMD:C_0402_1005Metric" H 3550 2950 50  0001 C CNN
@@
 AR Path="/5CE92455/5CDD1CD9" Ref="U4"  Part="1"
 AR Path="/5CDD1CD9" Ref="U4"  Part="1"
-F 0 "U1" V 6050 3600 60  0000 C CNN
+F 0 "U2" V 6050 3600 60  0000 C CNN
 F 1 "AD7779" V 5950 3600 60  0000 C CNN
 F 2 "QFN64:QFN-64-1EP_9x9mm_P0.5mm_EP7.3x7.3mm_ThermalVias" H 6000 3600 60  0001 C CNN
@@
 AR Path="/5CE92453/5CDD1CE0" Ref="J9"  Part="1"
 AR Path="/5CE92455/5CDD1CE0" Ref="J13"  Part="1"
-F 0 "J1" H 50  2925 50  0000 C CNN
+F 0 "J5" H 50  2925 50  0000 C CNN
 F 1 "Conn_02x08_Odd_Even" H 50  3016 50  0000 C CNN
 F 2 "Connector_PinHeader_2.54mm:PinHeader_2x08_P2.54mm_Vertical" H 0   3550 50  0001 C CNN
@@
 AR Path="/5CE92453/5CDD1CE7" Ref="J10"  Part="1"
 AR Path="/5CE92455/5CDD1CE7" Ref="J14"  Part="1"
-F 0 "J2" H 50  3975 50  0000 C CNN
+F 0 "J6" H 50  3975 50  0000 C CNN
 F 1 "Conn_02x08_Odd_Even" H 50  4066 50  0000 C CNN
 F 2 "Connector_PinHeader_2.54mm:PinHeader_2x08_P2.54mm_Vertical" H 0   4600 50  0001 C CNN
@@
 AR Path="/5CE92453/5CDD1CEE" Ref="J11"  Part="1"
 AR Path="/5CE92455/5CDD1CEE" Ref="J15"  Part="1"
-F 0 "J3" H 11600 3525 50  0000 C CNN
+F 0 "J7" H 11600 3525 50  0000 C CNN
 F 1 "Conn_02x08_Odd_Even" H 11600 3616 50  0000 C CNN
 F 2 "Connector_PinHeader_2.54mm:PinHeader_2x08_P2.54mm_Vertical" H 11550 4150 50  0001 C CNN
@@
 AR Path="/5CE92453/5CDD1CF5" Ref="J12"  Part="1"
 AR Path="/5CE92455/5CDD1CF5" Ref="J16"  Part="1"
-F 0 "J4" H 11600 2475 50  0000 C CNN
+F 0 "J8" H 11600 2475 50  0000 C CNN
 F 1 "Conn_02x08_Odd_Even" H 11600 2566 50  0000 C CNN
 F 2 "Connector_PinHeader_2.54mm:PinHeader_2x08_P2.54mm_Vertical" H 11550 3100 50  0001 C CNN
@@
 AR Path="/5CE92453/5CDD1D19" Ref="C46"  Part="1"
 AR Path="/5CE92455/5CDD1D19" Ref="C67"  Part="1"
-F 0 "C4" H 3642 3496 50  0000 L CNN
+F 0 "C25" H 3642 3496 50  0000 L CNN
 F 1 "1u" H 3642 3405 50  0000 L CNN
 F 2 "Capacitor_SMD:C_0402_1005Metric" H 3550 3450 50  0001 C CNN
@@
 AR Path="/5CE92453/5CDD1D24" Ref="C47"  Part="1"
 AR Path="/5CE92455/5CDD1D24" Ref="C68"  Part="1"
-F 0 "C5" H 3292 4496 50  0000 L CNN
+F 0 "C26" H 3292 4496 50  0000 L CNN
 F 1 "100n" H 3292 4405 50  0000 L CNN
 F 2 "Capacitor_SMD:C_0603_1608Metric" H 3200 4450 50  0001 C CNN
@@
 AR Path="/5CE92453/5CDD1D2B" Ref="C49"  Part="1"
 AR Path="/5CE92455/5CDD1D2B" Ref="C70"  Part="1"
-F 0 "C7" H 3292 3996 50  0000 L CNN
+F 0 "C28" H 3292 3996 50  0000 L CNN
 F 1 "100n" H 3292 3905 50  0000 L CNN
 F 2 "Capacitor_SMD:C_0402_1005Metric" H 3200 3950 50  0001 C CNN
@@
 AR Path="/5CE92453/5CDD1D32" Ref="C48"  Part="1"
 AR Path="/5CE92455/5CDD1D32" Ref="C69"  Part="1"
-F 0 "C6" H 3642 4496 50  0000 L CNN
+F 0 "C27" H 3642 4496 50  0000 L CNN
 F 1 "1u" H 3642 4405 50  0000 L CNN
 F 2 "Capacitor_SMD:C_0603_1608Metric" H 3550 4450 50  0001 C CNN
@@
 AR Path="/5CE92453/5CDD1D41" Ref="C50"  Part="1"
 AR Path="/5CE92455/5CDD1D41" Ref="C71"  Part="1"
-F 0 "C8" H 3642 3996 50  0000 L CNN
+F 0 "C29" H 3642 3996 50  0000 L CNN
 F 1 "1u" H 3642 3905 50  0000 L CNN
 F 2 "Capacitor_SMD:C_0402_1005Metric" H 3550 3950 50  0001 C CNN
@@
 AR Path="/5CE92453/5CDD1D4D" Ref="C53"  Part="1"
 AR Path="/5CE92455/5CDD1D4D" Ref="C74"  Part="1"
-F 0 "C11" H 8792 4296 50  0000 L CNN
+F 0 "C32" H 8792 4296 50  0000 L CNN
 F 1 "100n" H 8792 4205 50  0000 L CNN
 F 2 "Capacitor_SMD:C_0402_1005Metric" H 8700 4250 50  0001 C CNN
@@
 AR Path="/5CE92453/5CDD1D54" Ref="C51"  Part="1"
 AR Path="/5CE92455/5CDD1D54" Ref="C72"  Part="1"
-F 0 "C9" H 8792 4596 50  0000 L CNN
+F 0 "C30" H 8792 4596 50  0000 L CNN
 F 1 "100n" H 8792 4505 50  0000 L CNN
 F 2 "Capacitor_SMD:C_0402_1005Metric" H 8700 4550 50  0001 C CNN
@@
 AR Path="/5CE92453/5CDD1D5B" Ref="C54"  Part="1"
 AR Path="/5CE92455/5CDD1D5B" Ref="C75"  Part="1"
-F 0 "C12" H 8442 4296 50  0000 L CNN
+F 0 "C33" H 8442 4296 50  0000 L CNN
 F 1 "1u" H 8442 4205 50  0000 L CNN
 F 2 "Capacitor_SMD:C_0402_1005Metric" H 8350 4250 50  0001 C CNN
@@
 AR Path="/5CE92453/5CDD1D6A" Ref="C52"  Part="1"
 AR Path="/5CE92455/5CDD1D6A" Ref="C73"  Part="1"
-F 0 "C10" H 8442 4596 50  0000 L CNN
+F 0 "C31" H 8442 4596 50  0000 L CNN
 F 1 "1u" H 8442 4505 50  0000 L CNN
 F 2 "Capacitor_SMD:C_0402_1005Metric" H 8350 4550 50  0001 C CNN
@@
 AR Path="/5CE92453/5CDD1D75" Ref="C62"  Part="1"
 AR Path="/5CE92455/5CDD1D75" Ref="C83"  Part="1"
-F 0 "C20" H 8792 2496 50  0000 L CNN
+F 0 "C41" H 8792 2496 50  0000 L CNN
 F 1 "100n" H 8792 2405 50  0000 L CNN
 F 2 "Capacitor_SMD:C_0402_1005Metric" H 8700 2450 50  0001 C CNN
@@
 AR Path="/5CE92453/5CDD1D7C" Ref="C63"  Part="1"
 AR Path="/5CE92455/5CDD1D7C" Ref="C84"  Part="1"
-F 0 "C21" H 8442 2496 50  0000 L CNN
+F 0 "C42" H 8442 2496 50  0000 L CNN
 F 1 "1u" H 8442 2405 50  0000 L CNN
 F 2 "Capacitor_SMD:C_0402_1005Metric" H 8350 2450 50  0001 C CNN
@@
 AR Path="/5CE92453/5CDD1D89" Ref="C59"  Part="1"
 AR Path="/5CE92455/5CDD1D89" Ref="C80"  Part="1"
-F 0 "C17" H 8792 3096 50  0000 L CNN
+F 0 "C38" H 8792 3096 50  0000 L CNN
 F 1 "100n" H 8792 3005 50  0000 L CNN
 F 2 "Capacitor_SMD:C_0603_1608Metric" H 8700 3050 50  0001 C CNN
@@
 AR Path="/5CE92453/5CDD1D90" Ref="C60"  Part="1"
 AR Path="/5CE92455/5CDD1D90" Ref="C81"  Part="1"
-F 0 "C18" H 8442 3096 50  0000 L CNN
+F 0 "C39" H 8442 3096 50  0000 L CNN
 F 1 "1u" H 8442 3005 50  0000 L CNN
 F 2 "Capacitor_SMD:C_0603_1608Metric" H 8350 3050 50  0001 C CNN
@@
 AR Path="/5CE92453/5CDD1D9D" Ref="C61"  Part="1"
 AR Path="/5CE92455/5CDD1D9D" Ref="C82"  Part="1"
-F 0 "C19" H 8442 2796 50  0000 L CNN
+F 0 "C40" H 8442 2796 50  0000 L CNN
 F 1 "100n" H 8442 2705 50  0000 L CNN
 F 2 "Capacitor_SMD:C_0402_1005Metric" H 8350 2750 50  0001 C CNN
@@
 AR Path="/5CE92453/5CDD1DA7" Ref="C57"  Part="1"
 AR Path="/5CE92455/5CDD1DA7" Ref="C78"  Part="1"
-F 0 "C15" H 8792 3396 50  0000 L CNN
+F 0 "C36" H 8792 3396 50  0000 L CNN
 F 1 "100n" H 8792 3305 50  0000 L CNN
 F 2 "Capacitor_SMD:C_0603_1608Metric" H 8700 3350 50  0001 C CNN
@@
 AR Path="/5CE92453/5CDD1DAE" Ref="C58"  Part="1"
 AR Path="/5CE92455/5CDD1DAE" Ref="C79"  Part="1"
-F 0 "C16" H 8442 3396 50  0000 L CNN
+F 0 "C37" H 8442 3396 50  0000 L CNN
 F 1 "1u" H 8442 3305 50  0000 L CNN
 F 2 "Capacitor_SMD:C_0603_1608Metric" H 8350 3350 50  0001 C CNN
@@
 AR Path="/5CE92453/5CDD1DBB" Ref="C56"  Part="1"
 AR Path="/5CE92455/5CDD1DBB" Ref="C77"  Part="1"
-F 0 "C14" H 8442 3696 50  0000 L CNN
+F 0 "C35" H 8442 3696 50  0000 L CNN
 F 1 "100n" H 8442 3605 50  0000 L CNN
 F 2 "Capacitor_SMD:C_0402_1005Metric" H 8350 3650 50  0001 C CNN
@@
 AR Path="/5CE92453/5CDD1DC4" Ref="C55"  Part="1"
 AR Path="/5CE92455/5CDD1DC4" Ref="C76"  Part="1"
-F 0 "C13" H 8442 3996 50  0000 L CNN
+F 0 "C34" H 8442 3996 50  0000 L CNN
 F 1 "100n" H 8442 3905 50  0000 L CNN
 F 2 "Capacitor_SMD:C_0402_1005Metric" H 8350 3950 50  0001 C CNN
@@
 AR Path="/5CE92453/92BE555A" Ref="J55"  Part="1"
 AR Path="/5CE92455/92BE555A" Ref="J56"  Part="1"
-F 0 "J53" H 5900 1767 50  0000 C CNN
+F 0 "J54" H 5900 1767 50  0000 C CNN
 F 1 "Conn_02x10_Odd_Even" H 5900 1676 50  0000 C CNN
 F 2 "Connector_PinHeader_2.54mm:PinHeader_2x10_P2.54mm_Horizontal" H 5850 1150 50  0001 C CNN

Commit message: Add files via upload
Changed lines of the file:
@@
 $Descr A4 11693 8268
 encoding utf-8
-Sheet 2 22
+Sheet 5 22
 Title ""
 Date ""
@@
 AR Path="/5CE92453/5CDD1CC4" Ref="C43"  Part="1"
 AR Path="/5CE92455/5CDD1CC4" Ref="C64"  Part="1"
-F 0 "C22" H 3292 2996 50  0000 L CNN
+F 0 "C64" H 3292 2996 50  0000 L CNN
 F 1 "100n" H 3292 2905 50  0000 L CNN
 F 2 "Capacitor_SMD:C_0402_1005Metric" H 3200 2950 50  0001 C CNN
@@
 AR Path="/5CE92453/5CDD1CCB" Ref="C45"  Part="1"
 AR Path="/5CE92455/5CDD1CCB" Ref="C66"  Part="1"
-F 0 "C24" H 3292 3496 50  0000 L CNN
+F 0 "C66" H 3292 3496 50  0000 L CNN
 F 1 "100n" H 3292 3405 50  0000 L CNN
 F 2 "Capacitor_SMD:C_0402_1005Metric" H 3200 3450 50  0001 C CNN
@@
 AR Path="/5CE92453/5CDD1CD2" Ref="C44"  Part="1"
 AR Path="/5CE92455/5CDD1CD2" Ref="C65"  Part="1"
-F 0 "C23" H 3642 2996 50  0000 L CNN
+F 0 "C65" H 3642 2996 50  0000 L CNN
 F 1 "1u" H 3642 2905 50  0000 L CNN
 F 2 "Capacitor_SMD:C_0402_1005Metric" H 3550 2950 50  0001 C CNN
@@
 AR Path="/5CE92455/5CDD1CD9" Ref="U4"  Part="1"
 AR Path="/5CDD1CD9" Ref="U4"  Part="1"
-F 0 "U2" V 6050 3600 60  0000 C CNN
+F 0 "U4" V 6050 3600 60  0000 C CNN
 F 1 "AD7779" V 5950 3600 60  0000 C CNN
 F 2 "QFN64:QFN-64-1EP_9x9mm_P0.5mm_EP7.3x7.3mm_ThermalVias" H 6000 3600 60  0001 C CNN
@@
 AR Path="/5CE92453/5CDD1CE0" Ref="J9"  Part="1"
 AR Path="/5CE92455/5CDD1CE0" Ref="J13"  Part="1"
-F 0 "J5" H 50  2925 50  0000 C CNN
+F 0 "J13" H 50  2925 50  0000 C CNN
 F 1 "Conn_02x08_Odd_Even" H 50  3016 50  0000 C CNN
 F 2 "Connector_PinHeader_2.54mm:PinHeader_2x08_P2.54mm_Vertical" H 0   3550 50  0001 C CNN
@@
 AR Path="/5CE92453/5CDD1CE7" Ref="J10"  Part="1"
 AR Path="/5CE92455/5CDD1CE7" Ref="J14"  Part="1"
-F 0 "J6" H 50  3975 50  0000 C CNN
+F 0 "J14" H 50  3975 50  0000 C CNN
 F 1 "Conn_02x08_Odd_Even" H 50  4066 50  0000 C CNN
 F 2 "Connector_PinHeader_2.54mm:PinHeader_2x08_P2.54mm_Vertical" H 0   4600 50  0001 C CNN
@@
 AR Path="/5CE92453/5CDD1CEE" Ref="J11"  Part="1"
 AR Path="/5CE92455/5CDD1CEE" Ref="J15"  Part="1"
-F 0 "J7" H 11600 3525 50  0000 C CNN
+F 0 "J15" H 11600 3525 50  0000 C CNN
 F 1 "Conn_02x08_Odd_Even" H 11600 3616 50  0000 C CNN
 F 2 "Connector_PinHeader_2.54mm:PinHeader_2x08_P2.54mm_Vertical" H 11550 4150 50  0001 C CNN
@@
 AR Path="/5CE92453/5CDD1CF5" Ref="J12"  Part="1"
 AR Path="/5CE92455/5CDD1CF5" Ref="J16"  Part="1"
-F 0 "J8" H 11600 2475 50  0000 C CNN
+F 0 "J16" H 11600 2475 50  0000 C CNN
 F 1 "Conn_02x08_Odd_Even" H 11600 2566 50  0000 C CNN
 F 2 "Connector_PinHeader_2.54mm:PinHeader_2x08_P2.54mm_Vertical" H 11550 3100 50  0001 C CNN
@@
 AR Path="/5CE92453/5CDD1D19" Ref="C46"  Part="1"
 AR Path="/5CE92455/5CDD1D19" Ref="C67"  Part="1"
-F 0 "C25" H 3642 3496 50  0000 L CNN
+F 0 "C67" H 3642 3496 50  0000 L CNN
 F 1 "1u" H 3642 3405 50  0000 L CNN
 F 2 "Capacitor_SMD:C_0402_1005Metric" H 3550 3450 50  0001 C CNN
@@
 AR Path="/5CE92453/5CDD1D24" Ref="C47"  Part="1"
 AR Path="/5CE92455/5CDD1D24" Ref="C68"  Part="1"
-F 0 "C26" H 3292 4496 50  0000 L CNN
+F 0 "C68" H 3292 4496 50  0000 L CNN
 F 1 "100n" H 3292 4405 50  0000 L CNN
 F 2 "Capacitor_SMD:C_0603_1608Metric" H 3200 4450 50  0001 C CNN
@@
 AR Path="/5CE92453/5CDD1D2B" Ref="C49"  Part="1"
 AR Path="/5CE92455/5CDD1D2B" Ref="C70"  Part="1"
-F 0 "C28" H 3292 3996 50  0000 L CNN
+F 0 "C70" H 3292 3996 50  0000 L CNN
 F 1 "100n" H 3292 3905 50  0000 L CNN
 F 2 "Capacitor_SMD:C_0402_1005Metric" H 3200 3950 50  0001 C CNN
@@
 AR Path="/5CE92453/5CDD1D32" Ref="C48"  Part="1"
 AR Path="/5CE92455/5CDD1D32" Ref="C69"  Part="1"
-F 0 "C27" H 3642 4496 50  0000 L CNN
+F 0 "C69" H 3642 4496 50  0000 L CNN
 F 1 "1u" H 3642 4405 50  0000 L CNN
 F 2 "Capacitor_SMD:C_0603_1608Metric" H 3550 4450 50  0001 C CNN
@@
 AR Path="/5CE92453/5CDD1D41" Ref="C50"  Part="1"
 AR Path="/5CE92455/5CDD1D41" Ref="C71"  Part="1"
-F 0 "C29" H 3642 3996 50  0000 L CNN
+F 0 "C71" H 3642 3996 50  0000 L CNN
 F 1 "1u" H 3642 3905 50  0000 L CNN
 F 2 "Capacitor_SMD:C_0402_1005Metric" H 3550 3950 50  0001 C CNN
@@
 AR Path="/5CE92453/5CDD1D4D" Ref="C53"  Part="1"
 AR Path="/5CE92455/5CDD1D4D" Ref="C74"  Part="1"
-F 0 "C32" H 8792 4296 50  0000 L CNN
+F 0 "C74" H 8792 4296 50  0000 L CNN
 F 1 "100n" H 8792 4205 50  0000 L CNN
 F 2 "Capacitor_SMD:C_0402_1005Metric" H 8700 4250 50  0001 C CNN
@@
 AR Path="/5CE92453/5CDD1D54" Ref="C51"  Part="1"
 AR Path="/5CE92455/5CDD1D54" Ref="C72"  Part="1"
-F 0 "C30" H 8792 4596 50  0000 L CNN
+F 0 "C72" H 8792 4596 50  0000 L CNN
 F 1 "100n" H 8792 4505 50  0000 L CNN
 F 2 "Capacitor_SMD:C_0402_1005Metric" H 8700 4550 50  0001 C CNN
@@
 AR Path="/5CE92453/5CDD1D5B" Ref="C54"  Part="1"
 AR Path="/5CE92455/5CDD1D5B" Ref="C75"  Part="1"
-F 0 "C33" H 8442 4296 50  0000 L CNN
+F 0 "C75" H 8442 4296 50  0000 L CNN
 F 1 "1u" H 8442 4205 50  0000 L CNN
 F 2 "Capacitor_SMD:C_0402_1005Metric" H 8350 4250 50  0001 C CNN
@@
 AR Path="/5CE92453/5CDD1D6A" Ref="C52"  Part="1"
 AR Path="/5CE92455/5CDD1D6A" Ref="C73"  Part="1"
-F 0 "C31" H 8442 4596 50  0000 L CNN
+F 0 "C73" H 8442 4596 50  0000 L CNN
 F 1 "1u" H 8442 4505 50  0000 L CNN
 F 2 "Capacitor_SMD:C_0402_1005Metric" H 8350 4550 50  0001 C CNN
@@
 AR Path="/5CE92453/5CDD1D75" Ref="C62"  Part="1"
 AR Path="/5CE92455/5CDD1D75" Ref="C83"  Part="1"
-F 0 "C41" H 8792 2496 50  0000 L CNN
+F 0 "C83" H 8792 2496 50  0000 L CNN
 F 1 "100n" H 8792 2405 50  0000 L CNN
 F 2 "Capacitor_SMD:C_0402_1005Metric" H 8700 2450 50  0001 C CNN
@@
 AR Path="/5CE92453/5CDD1D7C" Ref="C63"  Part="1"
 AR Path="/5CE92455/5CDD1D7C" Ref="C84"  Part="1"
-F 0 "C42" H 8442 2496 50  0000 L CNN
+F 0 "C84" H 8442 2496 50  0000 L CNN
 F 1 "1u" H 8442 2405 50  0000 L CNN
 F 2 "Capacitor_SMD:C_0402_1005Metric" H 8350 2450 50  0001 C CNN
@@
 AR Path="/5CE92453/5CDD1D89" Ref="C59"  Part="1"
 AR Path="/5CE92455/5CDD1D89" Ref="C80"  Part="1"
-F 0 "C38" H 8792 3096 50  0000 L CNN
+F 0 "C80" H 8792 3096 50  0000 L CNN
 F 1 "100n" H 8792 3005 50  0000 L CNN
 F 2 "Capacitor_SMD:C_0603_1608Metric" H 8700 3050 50  0001 C CNN
@@
 AR Path="/5CE92453/5CDD1D90" Ref="C60"  Part="1"
 AR Path="/5CE92455/5CDD1D90" Ref="C81"  Part="1"
-F 0 "C39" H 8442 3096 50  0000 L CNN
+F 0 "C81" H 8442 3096 50  0000 L CNN
 F 1 "1u" H 8442 3005 50  0000 L CNN
 F 2 "Capacitor_SMD:C_0603_1608Metric" H 8350 3050 50  0001 C CNN
@@
 AR Path="/5CE92453/5CDD1D9D" Ref="C61"  Part="1"
 AR Path="/5CE92455/5CDD1D9D" Ref="C82"  Part="1"
-F 0 "C40" H 8442 2796 50  0000 L CNN
+F 0 "C82" H 8442 2796 50  0000 L CNN
 F 1 "100n" H 8442 2705 50  0000 L CNN
 F 2 "Capacitor_SMD:C_0402_1005Metric" H 8350 2750 50  0001 C CNN
@@
 AR Path="/5CE92453/5CDD1DA7" Ref="C57"  Part="1"
 AR Path="/5CE92455/5CDD1DA7" Ref="C78"  Part="1"
-F 0 "C36" H 8792 3396 50  0000 L CNN
+F 0 "C78" H 8792 3396 50  0000 L CNN
 F 1 "100n" H 8792 3305 50  0000 L CNN
 F 2 "Capacitor_SMD:C_0603_1608Metric" H 8700 3350 50  0001 C CNN
@@
 AR Path="/5CE92453/5CDD1DAE" Ref="C58"  Part="1"
 AR Path="/5CE92455/5CDD1DAE" Ref="C79"  Part="1"
-F 0 "C37" H 8442 3396 50  0000 L CNN
+F 0 "C79" H 8442 3396 50  0000 L CNN
 F 1 "1u" H 8442 3305 50  0000 L CNN
 F 2 "Capacitor_SMD:C_0603_1608Metric" H 8350 3350 50  0001 C CNN
@@
 AR Path="/5CE92453/5CDD1DBB" Ref="C56"  Part="1"
 AR Path="/5CE92455/5CDD1DBB" Ref="C77"  Part="1"
-F 0 "C35" H 8442 3696 50  0000 L CNN
+F 0 "C77" H 8442 3696 50  0000 L CNN
 F 1 "100n" H 8442 3605 50  0000 L CNN
 F 2 "Capacitor_SMD:C_0402_1005Metric" H 8350 3650 50  0001 C CNN
@@
 AR Path="/5CE92453/5CDD1DC4" Ref="C55"  Part="1"
 AR Path="/5CE92455/5CDD1DC4" Ref="C76"  Part="1"
-F 0 "C34" H 8442 3996 50  0000 L CNN
+F 0 "C76" H 8442 3996 50  0000 L CNN
 F 1 "100n" H 8442 3905 50  0000 L CNN
 F 2 "Capacitor_SMD:C_0402_1005Metric" H 8350 3950 50  0001 C CNN
@@
 AR Path="/5CE92453/92BE555A" Ref="J55"  Part="1"
 AR Path="/5CE92455/92BE555A" Ref="J56"  Part="1"
-F 0 "J54" H 5900 1767 50  0000 C CNN
+F 0 "J56" H 5900 1767 50  0000 C CNN
 F 1 "Conn_02x10_Odd_Even" H 5900 1676 50  0000 C CNN
 F 2 "Connector_PinHeader_2.54mm:PinHeader_2x10_P2.54mm_Horizontal" H 5850 1150 50  0001 C CNN
