File: KiCAD/FreeEEG32-alpha1.5.kicad_pcb (KiCad board)
At the start: 4 copper layers, 70 x 70 mm, 183 parts, among them J37 USB_B_Micro, J51 USB_B_Micro, J53 Conn_02x10_Odd_Even, J54 Conn_02x10_Odd_Even, J55 Conn_02x10_Odd_Even, J56 Conn_02x10_Odd_Even, J57 Conn_02x03_Odd_Even, J58 Conn_02x03_Odd_Even, J59 Conn_01x03, J60 Conn_01x03, J61 Conn_01x02, J62 Conn_01x02, J63 Conn_01x02, J64 Conn_01x02, SW1 SW_Push, SW2 SW_Push, T1 da2303, U1 AD7779, U10 LP5907, U11 LSM6DS3, U12 SN6505A, U13 473521001, U17 ADuM3160, U18 ADUM1402BRWZ, U19 ISO7341c, U2 AD7779, U3 AD7779, U4 AD7779, U5 LP5907, U6 LP5907, U7 ADR4525, U8 FXO-SM7_OSC-SMD7050_short, U9 STM32F765ZITx, Y1 32768Hz, Y2 16MHz

Commit message: Add files via upload
Connections:
- net MCU_100_TIM1_CH1 renamed /MCU/100_PA8
- net MCU_117_SPI2_SCK renamed /MCU/117_PD3
- net MCU_123_SPI1_MOSI renamed /MCU/123_PD7
- net MCU_126_SPI1_SCK renamed /MCU/126_PG11
- net MCU_140_SPI2_NSS renamed /MCU/140_PB9
- net MCU_1_SPI4_SCK renamed /MCU/1_PE2
- net MCU_26_SAI2_FS_B renamed /MCU/26_PC0
- net MCU_49_SAI2_SD_B renamed /MCU/49_PF11
- net MCU_69_I2C2_SCL renamed /MCU/69_PB10
- net MCU_70_I2C2_SDA renamed /MCU/70_PB11

Commit message: Add files via upload
Parts:
- removed J59, J60: Conn_01x03, Connector_PinSocket_2.54mm:PinSocket_1x03_P2.54mm_Vertical
- added J65: Conn_01x02, Connector_PinSocket_2.54mm:PinSocket_1x02_P2.54mm_Vertical, F.Cu at (174.1, 109.5)
- added J69: Conn_01x02, Connector_PinSocket_2.54mm:PinSocket_1x02_P2.54mm_Vertical, F.Cu at (174.1, 90.5)
- added J73: Conn_01x02, Connector_PinSocket_2.54mm:PinSocket_1x02_P2.54mm_Vertical, F.Cu at (125.9, 90.5)
- added J78: Conn_01x02, Connector_PinSocket_2.54mm:PinSocket_1x02_P2.54mm_Vertical, F.Cu at (140.5, 124.1)
- added J79: Conn_01x02, Connector_PinSocket_2.54mm:PinSocket_1x02_P2.54mm_Vertical, F.Cu at (125.9, 109.5)
- added J80: Conn_01x02, Connector_PinSocket_2.54mm:PinSocket_1x02_P2.54mm_Vertical, F.Cu at (159.5, 124.1)
- added J81: Conn_01x02, Connector_PinSocket_2.54mm:PinSocket_1x02_P2.54mm_Vertical, F.Cu at (159.5, 75.9)
- added J82: Conn_02x02_Odd_Even, Connector_PinSocket_2.54mm:PinSocket_2x02_P2.54mm_Horizontal, F.Cu at (178.0, 116.0)
- added J83: Conn_02x02_Odd_Even, Connector_PinSocket_2.54mm:PinSocket_2x02_P2.54mm_Horizontal, F.Cu at (164.2, 129.8)
- added J85: Conn_01x02, Connector_PinSocket_2.54mm:PinSocket_1x02_P2.54mm_Vertical, F.Cu at (140.5, 75.9)
- added R114: 0, Resistor_SMD:R_0402_1005Metric, B.Cu at (157.6, 122.9)
- added R115: 0, Resistor_SMD:R_0402_1005Metric, B.Cu at (172.9, 107.6)
- added R116: 0, Resistor_SMD:R_0402_1005Metric, B.Cu at (172.9, 92.4)
- added R117: 0, Resistor_SMD:R_0402_1005Metric, B.Cu at (127.1, 92.4)
- J57, J58: footprint Connector_PinSocket_2.54mm:PinSocket_2x03_P2.54mm_Vertical -> Connector_PinSocket_2.54mm:PinSocket_2x03_P2.54mm_Horizontal
- J61, J62, J63, J64: footprint Connector_PinSocket_2.54mm:PinSocket_1x02_P2.54mm_Vertical -> Connector_PinSocket_2.54mm:PinSocket_2x01_P2.54mm_Horizontal
- moved J57 5.46 mm to (127.1, 78.9), turned to 315 degrees
- moved C130 1.44 mm to (164.5, 110.3)
- moved C106 1.33 mm to (163.7, 109.5)
- moved C98 0.63 mm to (140.2, 90.6)
- moved C122 0.54 mm to (140.9, 89.5)
- moved R109 0.54 mm to (139.6, 92.1)
- moved C91 0.48 mm to (155.1, 74.5)
- moved C92 0.48 mm to (155.1, 77.1)
- moved J58 0.38 mm to (132.5, 73.5)
- moved J61 0.15 mm to (167.9, 73.9), turned to 225 degrees
- moved J63 0.15 mm to (132.1, 126.1), turned to 45 degrees
- moved J64 0.15 mm to (123.9, 117.9), turned to 45 degrees
- moved J62 0.15 mm to (176.1, 82.1), turned to 225 degrees
- turned R108 to 45 degrees
- turned SW1 to 225 degrees
Connections:
- net /MCU/54_PF14 renamed MCU_54_PF14_I2C4_SCL
- net /MCU/55_PF15 renamed MCU_55_PF15_I2C4_SDA
- net /MCU/69_PB10 renamed MCU_69_PB10_I2C2_SCL
- net /MCU/70_PB11 renamed MCU_70_PB11_I2C2_SDA
- net MCU_111_SDMMC1_D2 renamed MCU_111_PC10_SDMMC1_D2
- net MCU_112_SDMMC1_D3 renamed MCU_112_PC11_SDMMC1_D3
- net MCU_113_SDMMC1_CK renamed MCU_113_PC12_SDMMC1_CK
- net MCU_116_SDMMC1_CMD renamed MCU_116_PD2_SDMMC1_CMD
- net MCU_48_BOOT1 renamed MCU_48_PB2_BOOT1
- net MCU_97_SDMMC1_DETECT renamed MCU_97_PC7_SDMMC1_DETECT
- net MCU_98_SDMMC1_D0 renamed MCU_98_PC8_SDMMC1_D0
- net MCU_99_SDMMC1_D1 renamed MCU_99_PC9_SDMMC1_D1
- J37 pad 2: USB_POWER_2_D- -> /USB_POWER/2_D-
- J37 pad 3: USB_POWER_3_D+ -> /USB_POWER/3_D+
- J57 pad 1: ISO_SPI_2_GND1 -> ISO_SPI_5_INC
- J57 pad 2: ISO_SPI_1_VCC1 -> ISO_SPI_6_OUTD
- J57 pad 3: ISO_SPI_4_INB -> ISO_SPI_3_INA
- J57 pad 4: ISO_SPI_3_INA -> ISO_SPI_4_INB
- J57 pad 5: ISO_SPI_6_OUTD -> ISO_SPI_1_VCC1
- J57 pad 6: ISO_SPI_5_INC -> ISO_SPI_2_GND1
- J62 pad 1: USB_POWER_3_D+ -> POWER_2_VCC
- J62 pad 2: USB_POWER_2_D- -> POWER_1_GND
- U1 pad 14: ADC1_13_MODE0_GPIO0 -> ADC1_14_MODE1_GPIO1
- U1 pad 35: ADC1_34_SYNC_OUT -> ADC1_35_SYNC_IN
- U2 pad 35: ADC1_34_SYNC_OUT -> ADC1_35_SYNC_IN
- U3 pad 35: ADC1_34_SYNC_OUT -> ADC1_35_SYNC_IN
- U4 pad 35: ADC1_34_SYNC_OUT -> ADC1_35_SYNC_IN
- U8 pad 3: ADC1_32_XTAL2_MCLK -> CRYSTAL_3_OUT
- U8 pad 4: ADC1_24_IOVDD -> CRYSTAL_4_Vin
- U9 pad 10: /MCU/10_PF0 -> MCU_10_PF0_I2C2_SDA
- U9 pad 105: MCU_105_SYS_JTMS-SWDIO -> MCU_105_PA13_SYS_JTMS-SWDIO
- U9 pad 109: MCU_109_SYS_JTCK-SWCLK -> MCU_109_PA14_SYS_JTCK-SWCLK
- U9 pad 11: /MCU/11_PF1 -> MCU_11_PF1_I2C2_SCL
- U9 pad 22: /MCU/22_PF10 -> ADC3_30_DRDY
- U9 pad 5: ADC2_30_DRDY -> /MCU/5_PE6
- U9 pad 7: /MCU/7_PC13 -> ADC2_30_DRDY
- U9 pad 89: /MCU/89_PG4 -> ADC4_30_DRDY
- U9 pad 90: /MCU/90_PG5 -> ADC1_30_DRDY
Routing:
- net ADC1_35_SYNC_IN: track 0.00 -> 133.3 mm, vias 0 -> 4
- net MCU_48_PB2_BOOT1: track 2.54 -> 120.4 mm, vias 0 -> 4
- net ACC_5_VDDIO: track 330.7 -> 434.7 mm
- net ADC1_34_SYNC_OUT: track 99.2 -> 15.2 mm, vias 4 -> 1
- net MCU_105_PA13_SYS_JTMS-SWDIO: track 0.00 -> 42.6 mm, vias 0 -> 2
- net MCU_105_SYS_JTMS-SWDIO: track 40.0 -> 0.00 mm, vias 2 -> 0
- net AVDD_1_IN: track 122.1 -> 158.8 mm, vias 2 -> 5
- net ADC1_32_XTAL2_MCLK: track 53.2 -> 88.8 mm, vias 2 -> 3
- net ADC1_43_AVDD1B: track 358.0 -> 393.0 mm
- net AINREF-: track 203.5 -> 169.2 mm, vias 0 -> 3
- net POWER_1_GND: track 16.0 -> 49.9 mm
- net CRYSTAL_4_Vin: track 0.00 -> 29.4 mm, vias 0 -> 1
- net ADC1_24_IOVDD: track 267.7 -> 295.0 mm, vias 11 -> 10
- net POWER_2_VCC: track 23.6 -> 50.7 mm
- net CRYSTAL_3_OUT: track 0.00 -> 25.3 mm
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- added copper zone on In2.Cu, net ACC_6_GND
- removed copper zone on In2.Cu.GND, net ACC_6_GND
Other:
- board text added: "FreeEEG32+ alpha1.5"
- board text removed: "FreeEEG32 alpha1.5"

Commit message: Add files via upload
Parts:
- C113, C131, C132, R100, R99: moved to F.Cu
- moved C136 193.2 mm to (-24.3, -15.6), turned to 315 degrees
- moved C138 189.7 mm to (-15.6, -24.3), turned to 315 degrees
- moved C131 188.1 mm to (-22.2, 21.0), turned to 225 degrees
- moved C132 186.1 mm to (-21.0, 22.2), turned to 225 degrees
- moved J58 181.9 mm to (-22.9, -21.1)
- moved C107 180.7 mm to (7.11, 11.1), turned to 0 degrees
- moved C1 180.3 mm to (18.4, -4.57)
- moved C10 180.3 mm to (16.5, 3.45)
- moved C100 180.3 mm to (-6.35, -12.7)
- moved C101 180.3 mm to (-5.08, -13.3)
- moved C102 180.3 mm to (6.99, -12.1)
- moved C103 180.3 mm to (11.4, -7.49)
- moved C104 180.3 mm to (13.5, -5.65)
- moved C105 180.3 mm to (14.4, -4.76)
- moved C106 180.3 mm to (13.7, 9.53)
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Connections:
- net MCU_54_PF14_I2C4_SCL renamed /MCU/54_PF14
- net MCU_55_PF15_I2C4_SDA renamed /MCU/55_PF15
- net MCU_69_PB10_I2C2_SCL renamed /MCU/69_PB10
- net MCU_70_PB11_I2C2_SDA renamed /MCU/70_PB11
- C101 pad 1: ACC_5_VDDIO -> ACC_12_CS
- C102 pad 1: ACC_5_VDDIO -> ACC_12_CS
- C103 pad 1: ACC_5_VDDIO -> ACC_12_CS
- C105 pad 1: ACC_5_VDDIO -> ACC_12_CS
- C106 pad 1: ACC_5_VDDIO -> ACC_12_CS
- C107 pad 1: ACC_5_VDDIO -> ACC_12_CS
- C108 pad 1: ACC_5_VDDIO -> ACC_12_CS
- C110 pad 1: ACC_5_VDDIO -> ACC_12_CS
- C111 pad 1: ACC_5_VDDIO -> ACC_12_CS
- C112 pad 1: ACC_5_VDDIO -> ACC_12_CS
- C122 pad 1: ACC_5_VDDIO -> ACC_12_CS
- C127 pad 1: ACC_5_VDDIO -> ACC_12_CS
- C128 pad 1: ACC_5_VDDIO -> ACC_12_CS
- C129 pad 1: ACC_5_VDDIO -> ACC_12_CS
- C130 pad 1: ACC_5_VDDIO -> ACC_12_CS
- C133 pad 1: ACC_5_VDDIO -> ACC_12_CS
- C134 pad 1: ACC_5_VDDIO -> ACC_12_CS
- C135 pad 1: ISO_UART_1_VCC1 -> ACC_12_CS
- C135 pad 2: ISO_UART_2_GND1 -> ACC_6_GND
- C136 pad 1: ACC_5_VDDIO -> ISO_UART_16_VCC2
- C136 pad 2: ACC_6_GND -> ISO_UART_15_GND2
- C137 pad 1: ISO_SPI_1_VCC1 -> ACC_12_CS
- C137 pad 2: ISO_SPI_2_GND1 -> ACC_6_GND
- C138 pad 1: ACC_5_VDDIO -> ISO_SPI_16_VCC2
- C138 pad 2: ACC_6_GND -> ISO_SPI_15_GND2
- C93 pad 1: ACC_5_VDDIO -> ACC_12_CS
- C94 pad 1: ACC_5_VDDIO -> ACC_12_CS
- C95 pad 1: ACC_5_VDDIO -> ACC_12_CS
- C96 pad 1: ACC_5_VDDIO -> ACC_12_CS
- C97 pad 1: ACC_5_VDDIO -> ACC_12_CS
- C98 pad 1: ACC_5_VDDIO -> ACC_12_CS
- C99 pad 1: ACC_5_VDDIO -> ACC_12_CS
- J53 pad 2: /ADC1/57_VCM -> ADC1_57_VCM
- J54 pad 2: /ADC2/57_VCM -> ADC1_57_VCM
- J55 pad 2: /ADC3/57_VCM -> ADC1_57_VCM
- J56 pad 2: /ADC4/57_VCM -> ADC1_57_VCM
- J57 pad 1: ISO_SPI_5_INC -> ISO_SPI_16_VCC2
- J57 pad 2: ISO_SPI_6_OUTD -> ISO_SPI_15_GND2
- J57 pad 3: ISO_SPI_3_INA -> ISO_SPI_14_OUTA
- J57 pad 4: ISO_SPI_4_INB -> ISO_SPI_13_OUTB
- J57 pad 5: ISO_SPI_1_VCC1 -> ISO_SPI_12_OUTC
- J57 pad 6: ISO_SPI_2_GND1 -> ISO_SPI_11_IND
- J58 pad 1: ISO_UART_1_VCC1 -> ISO_UART_12_INC
- J58 pad 2: ISO_UART_2_GND1 -> ISO_UART_11_IND
- J58 pad 3: ISO_UART_3_INA -> ISO_UART_14_OUTA
- J58 pad 4: ISO_UART_4_INB -> ISO_UART_13_OUTB
- J58 pad 5: ISO_UART_5_OUTC -> ISO_UART_16_VCC2
- J58 pad 6: ISO_UART_6_OUTD -> ISO_UART_15_GND2
- J83 pad 3: ACC_5_VDDIO -> ACC_12_CS
- J85 pad 1: ACC_5_VDDIO -> ACC_12_CS
- SW1 pad 1: ACC_5_VDDIO -> ACC_12_CS
- U1 pad 57: /ADC1/57_VCM -> ADC1_57_VCM
- U10 pad 5: ACC_5_VDDIO -> ACC_12_CS
- U11 pad 5: ACC_5_VDDIO -> ACC_12_CS
- U11 pad 8: ACC_5_VDDIO -> ACC_12_CS
- U13 pad 4: ACC_5_VDDIO -> ACC_12_CS
- U17 pad 12: ACC_5_VDDIO -> ISO_USB_12_PIN
- U17 pad 13: ACC_5_VDDIO -> ACC_12_CS
- U17 pad 14: ACC_5_VDDIO -> ACC_12_CS
- U17 pad 16: ACC_5_VDDIO -> ACC_12_CS
- U18 pad 1: ISO_UART_1_VCC1 -> ACC_12_CS
- U18 pad 15: ACC_6_GND -> ISO_UART_15_GND2
- U18 pad 16: ACC_5_VDDIO -> ISO_UART_16_VCC2
- U18 pad 2: ISO_UART_2_GND1 -> ACC_6_GND
- U19 pad 1: ISO_SPI_1_VCC1 -> ACC_12_CS
- U19 pad 15: ACC_6_GND -> ISO_SPI_15_GND2
- U19 pad 16: ACC_5_VDDIO -> ISO_SPI_16_VCC2
- U19 pad 2: ISO_SPI_2_GND1 -> ACC_6_GND
- U2 pad 57: /ADC2/57_VCM -> ADC1_57_VCM
- U3 pad 57: /ADC3/57_VCM -> ADC1_57_VCM
- U4 pad 57: /ADC4/57_VCM -> ADC1_57_VCM
- U9 pad 101: ISO_UART_12_INC -> ISO_UART_4_INB
- U9 pad 102: ISO_UART_14_OUTA -> ISO_UART_6_OUTD
- U9 pad 103: ISO_UART_11_IND -> ISO_UART_5_OUTC
- U9 pad 104: ISO_UART_13_OUTB -> ISO_UART_3_INA
- U9 pad 108: ACC_5_VDDIO -> ACC_12_CS
- U9 pad 121: ACC_5_VDDIO -> ACC_12_CS
- U9 pad 131: ACC_5_VDDIO -> ACC_12_CS
- U9 pad 139: /MCU/139_PB8 -> ACC_4_INT1
- U9 pad 140: /MCU/140_PB9 -> ACC_1_SDO_SAO
- U9 pad 141: ACC_4_INT1 -> /MCU/141_PE0
- U9 pad 143: ACC_5_VDDIO -> ACC_12_CS
- U9 pad 144: ACC_5_VDDIO -> ACC_12_CS
- U9 pad 17: ACC_5_VDDIO -> ACC_12_CS
- U9 pad 19: /MCU/19_PF7 -> ISO_USB_12_PIN
- U9 pad 30: ACC_5_VDDIO -> ACC_12_CS
- U9 pad 32: ACC_5_VDDIO -> ACC_12_CS
- U9 pad 33: ACC_5_VDDIO -> ACC_12_CS
- U9 pad 39: ACC_5_VDDIO -> ACC_12_CS
- U9 pad 40: ISO_SPI_14_OUTA -> ISO_SPI_3_INA
- U9 pad 41: ISO_SPI_13_OUTB -> ISO_SPI_4_INB
- U9 pad 42: ISO_SPI_11_IND -> ISO_SPI_6_OUTD
- U9 pad 43: ISO_SPI_12_OUTC -> ISO_SPI_5_INC
- U9 pad 45: /MCU/45_PC5 -> ADC3_33_START
- U9 pad 46: ADC3_33_START -> ADC1_30_DRDY
- U9 pad 52: ACC_5_VDDIO -> ACC_12_CS
- U9 pad 6: ACC_5_VDDIO -> ACC_12_CS
- U9 pad 62: ACC_5_VDDIO -> ACC_12_CS
- U9 pad 72: ACC_5_VDDIO -> ACC_12_CS
- U9 pad 84: ACC_5_VDDIO -> ACC_12_CS
- U9 pad 90: ADC1_30_DRDY -> /MCU/90_PG5
- U9 pad 95: ACC_5_VDDIO -> ACC_12_CS
Routing:
- net ACC_5_VDDIO: track 434.7 -> 0.00 mm, vias 11 -> 0
- net ACC_12_CS: track 0.00 -> 341.6 mm, vias 0 -> 13
- net ADC1_57_VCM: track 0.00 -> 97.6 mm
- net AVDD_1_IN: track 158.8 -> 123.7 mm
- net ISO_UART_4_INB: track 6.92 -> 36.7 mm, vias 0 -> 1
- net ISO_UART_12_INC: track 32.4 -> 3.85 mm, vias 1 -> 0
- net ISO_UART_3_INA: track 3.85 -> 31.9 mm, vias 0 -> 1
- net ISO_UART_14_OUTA: track 31.7 -> 3.85 mm, vias 1 -> 0
- net ISO_UART_5_OUTC: track 3.85 -> 30.9 mm, vias 0 -> 1
- net ISO_UART_13_OUTB: track 32.0 -> 6.92 mm, vias 1 -> 0
- net ISO_UART_6_OUTD: track 6.92 -> 31.8 mm, vias 0 -> 1
- net ISO_UART_11_IND: track 31.6 -> 6.92 mm, vias 1 -> 0
- net /ADC4/57_VCM: track 24.4 -> 0.00 mm
- net /ADC3/57_VCM: track 24.4 -> 0.00 mm
- net /ADC2/57_VCM: track 24.4 -> 0.00 mm
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
Commit message: Add files via upload
Parts:
- added J88: Conn_01x02, Connector_PinSocket_2.54mm:PinSocket_1x02_P2.54mm_Vertical, F.Cu at (1.27, 24.8)
- added J89: Conn_01x02, Connector_PinSocket_2.54mm:PinSocket_1x02_P2.54mm_Vertical, F.Cu at (-24.8, 1.27)
- added J90: Conn_01x02, Connector_PinSocket_2.54mm:PinSocket_1x02_P2.54mm_Vertical, F.Cu at (24.8, -1.27)
- J65, J69, J73, J80: footprint Connector_PinSocket_2.54mm:PinSocket_1x02_P2.54mm_Vertical -> Connector_PinHeader_2.54mm:PinHeader_1x02_P2.54mm_Vertical
Routing:
- net ADC1_57_VCM: track 97.6 -> 283.9 mm, vias 0 -> 4
- net ADC1_24_IOVDD: track 300.1 -> 273.9 mm
- net ADC1_43_AVDD1B: track 397.7 -> 372.7 mm
- net AINREF-: track 169.2 -> 193.3 mm
- net ACC_12_CS: track 341.6 -> 317.9 mm
- net AVDD_1_IN: track 123.7 -> 104.2 mm, vias 5 -> 4
- net ADC1_32_XTAL2_MCLK: track 82.5 -> 93.6 mm
- net ADC1_35_SYNC_IN: track 128.7 -> 135.6 mm
- net MCU_48_PB2_BOOT1: track 120.8 -> 114.9 mm
- net ADC1_13_MODE0_GPIO0: track 186.2 -> 191.3 mm, vias 6 -> 7
- net /ADC3/49_REF_OUT: track 7.57 -> 4.10 mm
- net /MCU/114_PD0: track 3.02 -> 0.00 mm
- net ADC1_41_REF2+: track 187.8 -> 190.1 mm
- net /ADC3/51_AREG2CAP: track 5.16 -> 3.07 mm
- net /ADC3/59_AREG1CAP: track 5.55 -> 3.98 mm
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