File: KiCAD/ISO1.sch (KiCad schematic (older format))
At the start: 5 parts, among them J39 Conn_02x04_Odd_Even, J40 Conn_02x04_Odd_Even, U14 ISO7341c

Commit message: Add files via upload
Changed lines of the file:
@@
 AR Path="/637B2637/5CDC4527" Ref="U?"  Part="1"
 AR Path="/6385C8DD/5CDC4527" Ref="U?"  Part="1"
-F 0 "U14" H 3400 3547 60  0000 C CNN
+F 0 "U16" H 3400 3547 60  0000 C CNN
 F 1 "ISO7341c" H 3400 3441 60  0000 C CNN
 F 2 "Package_SO:SOIC-16W_7.5x10.3mm_P1.27mm" H 3400 2800 60  0001 C CNN
@@
 AR Path="/637B2637/75BAB1CD" Ref="C?"  Part="1"
 AR Path="/6385C8DD/75BAB1CD" Ref="C?"  Part="1"
-F 0 "C116" H 2292 2746 50  0000 L CNN
+F 0 "C120" H 2292 2746 50  0000 L CNN
 F 1 "100n" H 2292 2655 50  0000 L CNN
 F 2 "Capacitor_SMD:C_0402_1005Metric" H 2200 2700 50  0001 C CNN
@@
 AR Path="/637B2637/5CDC53E9" Ref="J?"  Part="1"
 AR Path="/6385C8DD/5CDC53E9" Ref="J?"  Part="1"
-F 0 "J39" H 2700 1667 50  0000 C CNN
+F 0 "J43" H 2700 1667 50  0000 C CNN
 F 1 "Conn_02x04_Odd_Even" H 2700 1576 50  0000 C CNN
 F 2 "Connector_PinHeader_2.54mm:PinHeader_2x04_P2.54mm_Vertical" H 2650 1350 50  0001 C CNN
@@
 AR Path="/637B2637/75BAB1D1" Ref="J?"  Part="1"
 AR Path="/6385C8DD/75BAB1D1" Ref="J?"  Part="1"
-F 0 "J40" H 4600 1617 50  0000 C CNN
+F 0 "J44" H 4600 1617 50  0000 C CNN
 F 1 "Conn_02x04_Odd_Even" H 4600 1526 50  0000 C CNN
 F 2 "Connector_PinHeader_2.54mm:PinHeader_2x04_P2.54mm_Vertical" H 4550 1300 50  0001 C CNN
@@
 AR Path="/637B2637/75BAB1D3" Ref="C?"  Part="1"
 AR Path="/6385C8DD/75BAB1D3" Ref="C?"  Part="1"
-F 0 "C117" H 4842 2696 50  0000 L CNN
+F 0 "C121" H 4842 2696 50  0000 L CNN
 F 1 "100n" H 4842 2605 50  0000 L CNN
 F 2 "Capacitor_SMD:C_0402_1005Metric" H 4750 2650 50  0001 C CNN
